Commit message: fix urdf coordinates and create two control example in python

File: universal_robot/ur_description/urdf/ur3_robot.urdf.xacro (robot description, xacro)
@@ -27,6 +27,6 @@
     </collision>
   </link>
-  <joint name="world_to_bar2" type="fixed">
-    <parent link="world"/>
+  <joint name="base_to_bar2" type="fixed">
+    <parent link="base_link"/>
     <child link="bar2"/>
     <origin xyz="0 0.038 -0.02" rpy="0 0 0"/>

Commit message: refine documents, add point cloud projects and python control

File: universal_robot/ur_description/urdf/ur3_robot.urdf.xacro (robot description, xacro)
@@ -30,5 +30,5 @@
     <parent link="base_link"/>
     <child link="bar2"/>
-    <origin xyz="0 0.038 -0.02" rpy="0 0 0"/>
+    <origin xyz="0 0.038 -0.02" rpy="0 0 1.57"/>
   </joint>
   <link name="bar1">

Commit message: added rg2 endeffector and, adjust controller_exec.py

File: universal_robot/ur_description/urdf/ur3_robot.urdf.xacro (robot description, xacro)
@@ -2,8 +2,18 @@
 <robot xmlns:xacro="http://wiki.ros.org/xacro"
        name="ur3" >
+    <property name="M_PI" value="3.14159265359" />
+    <property name="robot_prefix1" value=""/>
   <!-- ur3 -->
   <xacro:include filename="$(find ur_description)/urdf/ur3.urdf.xacro" />
   <!-- arm -->
   <xacro:ur3_robot prefix="" joint_limited="true"  />
+  <!-- arm extras
+  <xacro:include filename="$(find ur_description)/urdf/arm_extras_ur3.urdf.xacro" />-->
+  <!-- rg2 gripper -->
+  <xacro:include filename="$(find ur_description)/urdf/rg2.urdf.xacro" />
+  <!-- arm extras
+  <xacro:arm_extras prefix="${robot_prefix1}" joint_limited="true"/> -->
+  <!-- rg2 pipe -->
+  <xacro:rg2 prefix="${robot_prefix1}" joint_limited="true"/>
   <link name="world" />
   <joint name="world_joint" type="fixed">
@@ -63,5 +73,5 @@
     <collision>
       <geometry>
-        <box size="0.001 0.001 0.001"/>
+        <box size="0.8 1.0 0.02"/>
       </geometry>
     </collision>
